Commit message: fix robot jerk on start; adjust urdf for proper gravity compenstaiton; add 1khz control loop throttling (#42)

File: positronic/drivers/roboarm/kinova/model.urdf (robot description, URDF)
Before this commit: robot kinova_gen3, 10 links, 9 joints
Links:
- link tool_frame: mass None -> 0.74
